File: output/pcbs/crimes.kicad_pcb (KiCad board)
At the start: 2 copper layers, 277.5 x 100.4 mm, 148 parts

Commit message: Updated Mounting Holes
Parts:
- added _1: , MountingHole_2.2mm_M2_Pad_Via, F.Cu at (108.0, 97.0)
- added _2: , MountingHole_2.2mm_M2_Pad_Via, F.Cu at (186.0, 97.0)
- added _3: , MountingHole_2.2mm_M2_Pad_Via, F.Cu at (222.0, 97.0)
- added _4: , MountingHole_2.2mm_M2_Pad_Via, F.Cu at (87.4, 166.8)
- added _5: , MountingHole_2.2mm_M2_Pad_Via, F.Cu at (187.5, 152.2)
- added _6: , MountingHole_2.2mm_M2_Pad_Via, F.Cu at (223.5, 152.2)
- added _7: , MountingHole_2.2mm_M2_Pad_Via, F.Cu at (300.0, 97.0)
- added _8: , MountingHole_2.2mm_M2_Pad_Via, F.Cu at (318.0, 173.5)
Connections:
- MCU1 pad 1: row5 -> row3
- MCU1 pad 10: col13 -> col11
- MCU1 pad 11: col12 -> col10
- MCU1 pad 12: col11 -> col9
- MCU1 pad 13: col10 -> col8
- MCU1 pad 14: col9 -> P43
- MCU1 pad 15: col8 -> P42
- MCU1 pad 17: col7 -> P47
- MCU1 pad 2: row4 -> row2
- MCU1 pad 20: col6 -> P40
- MCU1 pad 21: col5 -> col7
- MCU1 pad 22: col4 -> col6
- MCU1 pad 23: col3 -> col5
- MCU1 pad 24: col2 -> col4
- MCU1 pad 25: col1 -> col3
- MCU1 pad 26: row1 -> col2
- MCU1 pad 27: R26 -> col1
- MCU1 pad 28: P27 -> row1
- MCU1 pad 4: row3 -> col15
- MCU1 pad 47: P14 -> row5
- MCU1 pad 48: P15 -> row4
- MCU1 pad 5: row2 -> P45
- MCU1 pad 6: col15 -> P44
- MCU1 pad 8: P32 -> col13
- MCU1 pad 9: P33 -> col12
Routing:
- net col13: track 126.8 -> 113.2 mm
- net col2: track 309.4 -> 317.9 mm
- net GND: track 104.7 -> 96.9 mm
- net col3: track 291.4 -> 297.5 mm
- net col1: track 323.8 -> 328.8 mm
- net col11: track 143.7 -> 148.1 mm
- net col9: track 157.9 -> 162.4 mm
- net col10: track 163.3 -> 167.5 mm
- net RST: track 18.1 -> 21.7 mm, vias 0 -> 2
- net col12: track 87.4 -> 90.5 mm
- net col8: track 193.9 -> 196.6 mm
- net row5: track 362.5 -> 365.1 mm
- net num_two: track 14.6 -> 12.1 mm
- net num_six: track 14.6 -> 12.1 mm
- net num_eight: track 14.6 -> 12.1 mm
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
Commit message: Updated Documentation.
Parts:
- moved B2 1.00 mm to (336.2, 110.6)
- moved ? 0.46 mm to (329.0, 111.6)
- moved ? 0.46 mm to (329.0, 109.6)
Routing:
- net VBUS: track 50.2 -> 51.2 mm
- net GND: track 96.9 -> 96.0 mm
Other:
- board text added: "JLCJLCJLCJLC"
