File: output/pcbs/switchplate.kicad_pcb (KiCad board)
At the start: 2 copper layers, 277.5 x 96.5 mm, 3 parts

Commit message: Updated Documentation.
Parts:
- added _1: , MountingHole_2.2mm_M2_Pad_Via, F.Cu at (108.0, 97.0)
- added _2: , MountingHole_2.2mm_M2_Pad_Via, F.Cu at (186.0, 97.0)
- added _3: , MountingHole_2.2mm_M2_Pad_Via, F.Cu at (222.0, 97.0)
- added _4: , MountingHole_2.2mm_M2_Pad_Via, F.Cu at (87.4, 166.8)
- added _5: , MountingHole_2.2mm_M2_Pad_Via, F.Cu at (187.5, 152.2)
- added _6: , MountingHole_2.2mm_M2_Pad_Via, F.Cu at (223.5, 152.2)
- added _7: , MountingHole_2.2mm_M2_Pad_Via, F.Cu at (300.0, 97.0)
- added _8: , MountingHole_2.2mm_M2_Pad_Via, F.Cu at (318.0, 173.5)

Commit message: Fixed MCU Pinout
Parts:
- moved _4 18.2 mm to (70.6, 159.8), turned to 90 degrees
- moved _1 1.00 mm to (108.0, 96.0)
- moved _2 1.00 mm to (186.0, 96.0)
- moved _3 1.00 mm to (222.0, 96.0)
- moved _5 1.00 mm to (187.5, 151.2)
- moved _6 1.00 mm to (223.5, 151.2)
- moved _7 1.00 mm to (300.0, 96.0)
- moved _8 1.00 mm to (318.0, 172.5)
Other:
- board size 277.5 x 96.5 mm -> 274.5 x 93.5 mm
- net class Default removed
- board text added: "JLCJLCJLCJLC"

Commit message: Fixed Pinouts.
Other:
- net class Default added: clearance 0.2, trace_width 0.25, via_dia 0.8, via_drill 0.4
- board text removed: "JLCJLCJLCJLC"
